Commit message: generating more URDFS

File: 75link_bf_1.urdf (robot description, URDF)
Before this commit: robot 55link_bf_2, 56 links, 55 joints
Links:
- added link link56, mass 1.5
- added link link57, mass 1.5
- added link link58, mass 1.5
- added link link59, mass 1.5
- added link link60, mass 1.5
- added link link61, mass 1.5
- added link link62, mass 1.5
- added link link63, mass 1.5
- added link link64, mass 1.5
- added link link65, mass 1.5
- added link link66, mass 1.5
- added link link67, mass 1.5
- added link link68, mass 1.5
- added link link69, mass 1.5
- added link link70, mass 1.5
- added link link71, mass 1.5
- added link link72, mass 1.5
- added link link73, mass 1.5
- added link link74, mass 1.5
- added link link75, mass 1.5
Joints:
- added joint joint56: type revolute, parent link55, child link56, origin xyz=55 0 0 rpy=0 0 0, axis 0 0 1, limit lower=0 upper=0 effort=0 velocity=0
- added joint joint57: type revolute, parent link56, child link57, origin xyz=56 0 0 rpy=0 0 0, axis 0 0 1, limit lower=0 upper=0 effort=0 velocity=0
- added joint joint58: type revolute, parent link57, child link58, origin xyz=57 0 0 rpy=0 0 0, axis 0 0 1, limit lower=0 upper=0 effort=0 velocity=0
- added joint joint59: type revolute, parent link58, child link59, origin xyz=58 0 0 rpy=0 0 0, axis 0 0 1, limit lower=0 upper=0 effort=0 velocity=0
- added joint joint60: type revolute, parent link59, child link60, origin xyz=59 0 0 rpy=0 0 0, axis 0 0 1, limit lower=0 upper=0 effort=0 velocity=0
- added joint joint61: type revolute, parent link60, child link61, origin xyz=60 0 0 rpy=0 0 0, axis 0 0 1, limit lower=0 upper=0 effort=0 velocity=0
- added joint joint62: type revolute, parent link61, child link62, origin xyz=61 0 0 rpy=0 0 0, axis 0 0 1, limit lower=0 upper=0 effort=0 velocity=0
- added joint joint63: type revolute, parent link62, child link63, origin xyz=62 0 0 rpy=0 0 0, axis 0 0 1, limit lower=0 upper=0 effort=0 velocity=0
- added joint joint64: type revolute, parent link63, child link64, origin xyz=63 0 0 rpy=0 0 0, axis 0 0 1, limit lower=0 upper=0 effort=0 velocity=0
- added joint joint65: type revolute, parent link64, child link65, origin xyz=64 0 0 rpy=0 0 0, axis 0 0 1, limit lower=0 upper=0 effort=0 velocity=0
- added joint joint66: type revolute, parent link65, child link66, origin xyz=65 0 0 rpy=0 0 0, axis 0 0 1, limit lower=0 upper=0 effort=0 velocity=0
- added joint joint67: type revolute, parent link66, child link67, origin xyz=66 0 0 rpy=0 0 0, axis 0 0 1, limit lower=0 upper=0 effort=0 velocity=0
- added joint joint68: type revolute, parent link67, child link68, origin xyz=67 0 0 rpy=0 0 0, axis 0 0 1, limit lower=0 upper=0 effort=0 velocity=0
- added joint joint69: type revolute, parent link68, child link69, origin xyz=68 0 0 rpy=0 0 0, axis 0 0 1, limit lower=0 upper=0 effort=0 velocity=0
- added joint joint70: type revolute, parent link69, child link70, origin xyz=69 0 0 rpy=0 0 0, axis 0 0 1, limit lower=0 upper=0 effort=0 velocity=0
- added joint joint71: type revolute, parent link70, child link71, origin xyz=70 0 0 rpy=0 0 0, axis 0 0 1, limit lower=0 upper=0 effort=0 velocity=0
- added joint joint72: type revolute, parent link71, child link72, origin xyz=71 0 0 rpy=0 0 0, axis 0 0 1, limit lower=0 upper=0 effort=0 velocity=0
- added joint joint73: type revolute, parent link72, child link73, origin xyz=72 0 0 rpy=0 0 0, axis 0 0 1, limit lower=0 upper=0 effort=0 velocity=0
- added joint joint74: type revolute, parent link73, child link74, origin xyz=73 0 0 rpy=0 0 0, axis 0 0 1, limit lower=0 upper=0 effort=0 velocity=0
- added joint joint75: type revolute, parent link74, child link75, origin xyz=74 0 0 rpy=0 0 0, axis 0 0 1, limit lower=0 upper=0 effort=0 velocity=0
- joint joint10: origin xyz=5 0 0 rpy=0 0 0 -> xyz=9 0 0 rpy=0 0 0; parent link5 -> link9
- joint joint11: origin xyz=5 0 0 rpy=0 0 0 -> xyz=10 0 0 rpy=0 0 0; parent link5 -> link10
- joint joint12: origin xyz=6 0 0 rpy=0 0 0 -> xyz=11 0 0 rpy=0 0 0; parent link6 -> link11
- joint joint13: origin xyz=6 0 0 rpy=0 0 0 -> xyz=12 0 0 rpy=0 0 0; parent link6 -> link12
- joint joint14: origin xyz=7 0 0 rpy=0 0 0 -> xyz=13 0 0 rpy=0 0 0; parent link7 -> link13
- joint joint15: origin xyz=7 0 0 rpy=0 0 0 -> xyz=14 0 0 rpy=0 0 0; parent link7 -> link14
- joint joint16: origin xyz=8 0 0 rpy=0 0 0 -> xyz=15 0 0 rpy=0 0 0; parent link8 -> link15
- joint joint17: origin xyz=8 0 0 rpy=0 0 0 -> xyz=16 0 0 rpy=0 0 0; parent link8 -> link16
- joint joint18: origin xyz=9 0 0 rpy=0 0 0 -> xyz=17 0 0 rpy=0 0 0; parent link9 -> link17
- joint joint19: origin xyz=9 0 0 rpy=0 0 0 -> xyz=18 0 0 rpy=0 0 0; parent link9 -> link18
- joint joint20: origin xyz=10 0 0 rpy=0 0 0 -> xyz=19 0 0 rpy=0 0 0; parent link10 -> link19
- joint joint21: origin xyz=10 0 0 rpy=0 0 0 -> xyz=20 0 0 rpy=0 0 0; parent link10 -> link20
- joint joint22: origin xyz=11 0 0 rpy=0 0 0 -> xyz=21 0 0 rpy=0 0 0; parent link11 -> link21
- joint joint23: origin xyz=11 0 0 rpy=0 0 0 -> xyz=22 0 0 rpy=0 0 0; parent link11 -> link22
- joint joint24: origin xyz=12 0 0 rpy=0 0 0 -> xyz=23 0 0 rpy=0 0 0; parent link12 -> link23
- joint joint25: origin xyz=12 0 0 rpy=0 0 0 -> xyz=24 0 0 rpy=0 0 0; parent link12 -> link24
- joint joint26: origin xyz=13 0 0 rpy=0 0 0 -> xyz=25 0 0 rpy=0 0 0; parent link13 -> link25
- joint joint27: origin xyz=13 0 0 rpy=0 0 0 -> xyz=26 0 0 rpy=0 0 0; parent link13 -> link26
- joint joint28: origin xyz=14 0 0 rpy=0 0 0 -> xyz=27 0 0 rpy=0 0 0; parent link14 -> link27
- joint joint29: origin xyz=14 0 0 rpy=0 0 0 -> xyz=28 0 0 rpy=0 0 0; parent link14 -> link28
- joint joint3: origin xyz=1 0 0 rpy=0 0 0 -> xyz=2 0 0 rpy=0 0 0; parent link1 -> link2
- joint joint30: origin xyz=15 0 0 rpy=0 0 0 -> xyz=29 0 0 rpy=0 0 0; parent link15 -> link29
- joint joint31: origin xyz=15 0 0 rpy=0 0 0 -> xyz=30 0 0 rpy=0 0 0; parent link15 -> link30
- joint joint32: origin xyz=16 0 0 rpy=0 0 0 -> xyz=31 0 0 rpy=0 0 0; parent link16 -> link31
- joint joint33: origin xyz=16 0 0 rpy=0 0 0 -> xyz=32 0 0 rpy=0 0 0; parent link16 -> link32
- joint joint34: origin xyz=17 0 0 rpy=0 0 0 -> xyz=33 0 0 rpy=0 0 0; parent link17 -> link33
- joint joint35: origin xyz=17 0 0 rpy=0 0 0 -> xyz=34 0 0 rpy=0 0 0; parent link17 -> link34
- joint joint36: origin xyz=18 0 0 rpy=0 0 0 -> xyz=35 0 0 rpy=0 0 0; parent link18 -> link35
- joint joint37: origin xyz=18 0 0 rpy=0 0 0 -> xyz=36 0 0 rpy=0 0 0; parent link18 -> link36
- joint joint38: origin xyz=19 0 0 rpy=0 0 0 -> xyz=37 0 0 rpy=0 0 0; parent link19 -> link37
- joint joint39: origin xyz=19 0 0 rpy=0 0 0 -> xyz=38 0 0 rpy=0 0 0; parent link19 -> link38
- joint joint4: origin xyz=2 0 0 rpy=0 0 0 -> xyz=3 0 0 rpy=0 0 0; parent link2 -> link3
- joint joint40: origin xyz=20 0 0 rpy=0 0 0 -> xyz=39 0 0 rpy=0 0 0; parent link20 -> link39
- joint joint41: origin xyz=20 0 0 rpy=0 0 0 -> xyz=40 0 0 rpy=0 0 0; parent link20 -> link40
- joint joint42: origin xyz=21 0 0 rpy=0 0 0 -> xyz=41 0 0 rpy=0 0 0; parent link21 -> link41
- joint joint43: origin xyz=21 0 0 rpy=0 0 0 -> xyz=42 0 0 rpy=0 0 0; parent link21 -> link42
- joint joint44: origin xyz=22 0 0 rpy=0 0 0 -> xyz=43 0 0 rpy=0 0 0; parent link22 -> link43
- joint joint45: origin xyz=22 0 0 rpy=0 0 0 -> xyz=44 0 0 rpy=0 0 0; parent link22 -> link44
- joint joint46: origin xyz=23 0 0 rpy=0 0 0 -> xyz=45 0 0 rpy=0 0 0; parent link23 -> link45
- joint joint47: origin xyz=23 0 0 rpy=0 0 0 -> xyz=46 0 0 rpy=0 0 0; parent link23 -> link46
- joint joint48: origin xyz=24 0 0 rpy=0 0 0 -> xyz=47 0 0 rpy=0 0 0; parent link24 -> link47
- joint joint49: origin xyz=24 0 0 rpy=0 0 0 -> xyz=48 0 0 rpy=0 0 0; parent link24 -> link48
- joint joint5: origin xyz=2 0 0 rpy=0 0 0 -> xyz=4 0 0 rpy=0 0 0; parent link2 -> link4
- joint joint50: origin xyz=25 0 0 rpy=0 0 0 -> xyz=49 0 0 rpy=0 0 0; parent link25 -> link49
- joint joint51: origin xyz=25 0 0 rpy=0 0 0 -> xyz=50 0 0 rpy=0 0 0; parent link25 -> link50
- joint joint52: origin xyz=26 0 0 rpy=0 0 0 -> xyz=51 0 0 rpy=0 0 0; parent link26 -> link51
- joint joint53: origin xyz=26 0 0 rpy=0 0 0 -> xyz=52 0 0 rpy=0 0 0; parent link26 -> link52
- joint joint54: origin xyz=27 0 0 rpy=0 0 0 -> xyz=53 0 0 rpy=0 0 0; parent link27 -> link53
- joint joint55: origin xyz=27 0 0 rpy=0 0 0 -> xyz=54 0 0 rpy=0 0 0; parent link27 -> link54
- joint joint6: origin xyz=3 0 0 rpy=0 0 0 -> xyz=5 0 0 rpy=0 0 0; parent link3 -> link5
- joint joint7: origin xyz=3 0 0 rpy=0 0 0 -> xyz=6 0 0 rpy=0 0 0; parent link3 -> link6
- joint joint8: origin xyz=4 0 0 rpy=0 0 0 -> xyz=7 0 0 rpy=0 0 0; parent link4 -> link7
- joint joint9: origin xyz=4 0 0 rpy=0 0 0 -> xyz=8 0 0 rpy=0 0 0; parent link4 -> link8

File: 75link_bf_2.urdf (robot description, URDF)
Before this commit: robot 55link_bf_5, 56 links, 55 joints
Links:
- added link link56, mass 1.5
- added link link57, mass 1.5
- added link link58, mass 1.5
- added link link59, mass 1.5
- added link link60, mass 1.5
- added link link61, mass 1.5
- added link link62, mass 1.5
- added link link63, mass 1.5
- added link link64, mass 1.5
- added link link65, mass 1.5
- added link link66, mass 1.5
- added link link67, mass 1.5
- added link link68, mass 1.5
- added link link69, mass 1.5
- added link link70, mass 1.5
- added link link71, mass 1.5
- added link link72, mass 1.5
- added link link73, mass 1.5
- added link link74, mass 1.5
- added link link75, mass 1.5
Joints:
- added joint joint56: type revolute, parent link28, child link56, origin xyz=28 0 0 rpy=0 0 0, axis 0 0 1, limit lower=0 upper=0 effort=0 velocity=0
- added joint joint57: type revolute, parent link28, child link57, origin xyz=28 0 0 rpy=0 0 0, axis 0 0 1, limit lower=0 upper=0 effort=0 velocity=0
- added joint joint58: type revolute, parent link29, child link58, origin xyz=29 0 0 rpy=0 0 0, axis 0 0 1, limit lower=0 upper=0 effort=0 velocity=0
- added joint joint59: type revolute, parent link29, child link59, origin xyz=29 0 0 rpy=0 0 0, axis 0 0 1, limit lower=0 upper=0 effort=0 velocity=0
- added joint joint60: type revolute, parent link30, child link60, origin xyz=30 0 0 rpy=0 0 0, axis 0 0 1, limit lower=0 upper=0 effort=0 velocity=0
- added joint joint61: type revolute, parent link30, child link61, origin xyz=30 0 0 rpy=0 0 0, axis 0 0 1, limit lower=0 upper=0 effort=0 velocity=0
- added joint joint62: type revolute, parent link31, child link62, origin xyz=31 0 0 rpy=0 0 0, axis 0 0 1, limit lower=0 upper=0 effort=0 velocity=0
- added joint joint63: type revolute, parent link31, child link63, origin xyz=31 0 0 rpy=0 0 0, axis 0 0 1, limit lower=0 upper=0 effort=0 velocity=0
- added joint joint64: type revolute, parent link32, child link64, origin xyz=32 0 0 rpy=0 0 0, axis 0 0 1, limit lower=0 upper=0 effort=0 velocity=0
- added joint joint65: type revolute, parent link32, child link65, origin xyz=32 0 0 rpy=0 0 0, axis 0 0 1, limit lower=0 upper=0 effort=0 velocity=0
- added joint joint66: type revolute, parent link33, child link66, origin xyz=33 0 0 rpy=0 0 0, axis 0 0 1, limit lower=0 upper=0 effort=0 velocity=0
- added joint joint67: type revolute, parent link33, child link67, origin xyz=33 0 0 rpy=0 0 0, axis 0 0 1, limit lower=0 upper=0 effort=0 velocity=0
- added joint joint68: type revolute, parent link34, child link68, origin xyz=34 0 0 rpy=0 0 0, axis 0 0 1, limit lower=0 upper=0 effort=0 velocity=0
- added joint joint69: type revolute, parent link34, child link69, origin xyz=34 0 0 rpy=0 0 0, axis 0 0 1, limit lower=0 upper=0 effort=0 velocity=0
- added joint joint70: type revolute, parent link35, child link70, origin xyz=35 0 0 rpy=0 0 0, axis 0 0 1, limit lower=0 upper=0 effort=0 velocity=0
- added joint joint71: type revolute, parent link35, child link71, origin xyz=35 0 0 rpy=0 0 0, axis 0 0 1, limit lower=0 upper=0 effort=0 velocity=0
- added joint joint72: type revolute, parent link36, child link72, origin xyz=36 0 0 rpy=0 0 0, axis 0 0 1, limit lower=0 upper=0 effort=0 velocity=0
- added joint joint73: type revolute, parent link36, child link73, origin xyz=36 0 0 rpy=0 0 0, axis 0 0 1, limit lower=0 upper=0 effort=0 velocity=0
- added joint joint74: type revolute, parent link37, child link74, origin xyz=37 0 0 rpy=0 0 0, axis 0 0 1, limit lower=0 upper=0 effort=0 velocity=0
- added joint joint75: type revolute, parent link37, child link75, origin xyz=37 0 0 rpy=0 0 0, axis 0 0 1, limit lower=0 upper=0 effort=0 velocity=0
- joint joint10: origin xyz=2 0 0 rpy=0 0 0 -> xyz=5 0 0 rpy=0 0 0; parent link2 -> link5
- joint joint11: origin xyz=2 0 0 rpy=0 0 0 -> xyz=5 0 0 rpy=0 0 0; parent link2 -> link5
- joint joint12: origin xyz=3 0 0 rpy=0 0 0 -> xyz=6 0 0 rpy=0 0 0; parent link3 -> link6
- joint joint13: origin xyz=3 0 0 rpy=0 0 0 -> xyz=6 0 0 rpy=0 0 0; parent link3 -> link6
- joint joint14: origin xyz=3 0 0 rpy=0 0 0 -> xyz=7 0 0 rpy=0 0 0; parent link3 -> link7
- joint joint15: origin xyz=3 0 0 rpy=0 0 0 -> xyz=7 0 0 rpy=0 0 0; parent link3 -> link7
- joint joint16: origin xyz=3 0 0 rpy=0 0 0 -> xyz=8 0 0 rpy=0 0 0; parent link3 -> link8
- joint joint17: origin xyz=4 0 0 rpy=0 0 0 -> xyz=8 0 0 rpy=0 0 0; parent link4 -> link8
- joint joint18: origin xyz=4 0 0 rpy=0 0 0 -> xyz=9 0 0 rpy=0 0 0; parent link4 -> link9
- joint joint19: origin xyz=4 0 0 rpy=0 0 0 -> xyz=9 0 0 rpy=0 0 0; parent link4 -> link9
- joint joint20: origin xyz=4 0 0 rpy=0 0 0 -> xyz=10 0 0 rpy=0 0 0; parent link4 -> link10
- joint joint21: origin xyz=4 0 0 rpy=0 0 0 -> xyz=10 0 0 rpy=0 0 0; parent link4 -> link10
- joint joint22: origin xyz=5 0 0 rpy=0 0 0 -> xyz=11 0 0 rpy=0 0 0; parent link5 -> link11
- joint joint23: origin xyz=5 0 0 rpy=0 0 0 -> xyz=11 0 0 rpy=0 0 0; parent link5 -> link11
- joint joint24: origin xyz=5 0 0 rpy=0 0 0 -> xyz=12 0 0 rpy=0 0 0; parent link5 -> link12
- joint joint25: origin xyz=5 0 0 rpy=0 0 0 -> xyz=12 0 0 rpy=0 0 0; parent link5 -> link12
- joint joint26: origin xyz=5 0 0 rpy=0 0 0 -> xyz=13 0 0 rpy=0 0 0; parent link5 -> link13
- joint joint27: origin xyz=6 0 0 rpy=0 0 0 -> xyz=13 0 0 rpy=0 0 0; parent link6 -> link13
- joint joint28: origin xyz=6 0 0 rpy=0 0 0 -> xyz=14 0 0 rpy=0 0 0; parent link6 -> link14
- joint joint29: origin xyz=6 0 0 rpy=0 0 0 -> xyz=14 0 0 rpy=0 0 0; parent link6 -> link14
- joint joint30: origin xyz=6 0 0 rpy=0 0 0 -> xyz=15 0 0 rpy=0 0 0; parent link6 -> link15
- joint joint31: origin xyz=6 0 0 rpy=0 0 0 -> xyz=15 0 0 rpy=0 0 0; parent link6 -> link15
- joint joint32: origin xyz=7 0 0 rpy=0 0 0 -> xyz=16 0 0 rpy=0 0 0; parent link7 -> link16
- joint joint33: origin xyz=7 0 0 rpy=0 0 0 -> xyz=16 0 0 rpy=0 0 0; parent link7 -> link16
- joint joint34: origin xyz=7 0 0 rpy=0 0 0 -> xyz=17 0 0 rpy=0 0 0; parent link7 -> link17
- joint joint35: origin xyz=7 0 0 rpy=0 0 0 -> xyz=17 0 0 rpy=0 0 0; parent link7 -> link17
- joint joint36: origin xyz=7 0 0 rpy=0 0 0 -> xyz=18 0 0 rpy=0 0 0; parent link7 -> link18
- joint joint37: origin xyz=8 0 0 rpy=0 0 0 -> xyz=18 0 0 rpy=0 0 0; parent link8 -> link18
- joint joint38: origin xyz=8 0 0 rpy=0 0 0 -> xyz=19 0 0 rpy=0 0 0; parent link8 -> link19
- joint joint39: origin xyz=8 0 0 rpy=0 0 0 -> xyz=19 0 0 rpy=0 0 0; parent link8 -> link19
- joint joint4: origin xyz=1 0 0 rpy=0 0 0 -> xyz=2 0 0 rpy=0 0 0; parent link1 -> link2
- joint joint40: origin xyz=8 0 0 rpy=0 0 0 -> xyz=20 0 0 rpy=0 0 0; parent link8 -> link20
- joint joint41: origin xyz=8 0 0 rpy=0 0 0 -> xyz=20 0 0 rpy=0 0 0; parent link8 -> link20
- joint joint42: origin xyz=9 0 0 rpy=0 0 0 -> xyz=21 0 0 rpy=0 0 0; parent link9 -> link21
- joint joint43: origin xyz=9 0 0 rpy=0 0 0 -> xyz=21 0 0 rpy=0 0 0; parent link9 -> link21
- joint joint44: origin xyz=9 0 0 rpy=0 0 0 -> xyz=22 0 0 rpy=0 0 0; parent link9 -> link22
- joint joint45: origin xyz=9 0 0 rpy=0 0 0 -> xyz=22 0 0 rpy=0 0 0; parent link9 -> link22
- joint joint46: origin xyz=9 0 0 rpy=0 0 0 -> xyz=23 0 0 rpy=0 0 0; parent link9 -> link23
- joint joint47: origin xyz=10 0 0 rpy=0 0 0 -> xyz=23 0 0 rpy=0 0 0; parent link10 -> link23
- joint joint48: origin xyz=10 0 0 rpy=0 0 0 -> xyz=24 0 0 rpy=0 0 0; parent link10 -> link24
- joint joint49: origin xyz=10 0 0 rpy=0 0 0 -> xyz=24 0 0 rpy=0 0 0; parent link10 -> link24
- joint joint5: origin xyz=1 0 0 rpy=0 0 0 -> xyz=2 0 0 rpy=0 0 0; parent link1 -> link2
- joint joint50: origin xyz=10 0 0 rpy=0 0 0 -> xyz=25 0 0 rpy=0 0 0; parent link10 -> link25
- joint joint51: origin xyz=10 0 0 rpy=0 0 0 -> xyz=25 0 0 rpy=0 0 0; parent link10 -> link25
- joint joint52: origin xyz=11 0 0 rpy=0 0 0 -> xyz=26 0 0 rpy=0 0 0; parent link11 -> link26
- joint joint53: origin xyz=11 0 0 rpy=0 0 0 -> xyz=26 0 0 rpy=0 0 0; parent link11 -> link26
- joint joint54: origin xyz=11 0 0 rpy=0 0 0 -> xyz=27 0 0 rpy=0 0 0; parent link11 -> link27
- joint joint55: origin xyz=11 0 0 rpy=0 0 0 -> xyz=27 0 0 rpy=0 0 0; parent link11 -> link27
- joint joint6: origin xyz=1 0 0 rpy=0 0 0 -> xyz=3 0 0 rpy=0 0 0; parent link1 -> link3
- joint joint7: origin xyz=2 0 0 rpy=0 0 0 -> xyz=3 0 0 rpy=0 0 0; parent link2 -> link3
- joint joint8: origin xyz=2 0 0 rpy=0 0 0 -> xyz=4 0 0 rpy=0 0 0; parent link2 -> link4
- joint joint9: origin xyz=2 0 0 rpy=0 0 0 -> xyz=4 0 0 rpy=0 0 0; parent link2 -> link4

File: 80link_bf_1.urdf (robot description, URDF)
Before this commit: robot 55link_bf_1, 56 links, 55 joints
Links:
- added link link56, mass 1.5
- added link link57, mass 1.5
- added link link58, mass 1.5
- added link link59, mass 1.5
- added link link60, mass 1.5
- added link link61, mass 1.5
- added link link62, mass 1.5
- added link link63, mass 1.5
- added link link64, mass 1.5
- added link link65, mass 1.5
- added link link66, mass 1.5
- added link link67, mass 1.5
- added link link68, mass 1.5
- added link link69, mass 1.5
- added link link70, mass 1.5
- added link link71, mass 1.5
- added link link72, mass 1.5
- added link link73, mass 1.5
- added link link74, mass 1.5
- added link link75, mass 1.5
- added link link76, mass 1.5
- added link link77, mass 1.5
- added link link78, mass 1.5
- added link link79, mass 1.5
- added link link80, mass 1.5
Joints:
- added joint joint56: type revolute, parent link55, child link56, origin xyz=55 0 0 rpy=0 0 0, axis 0 0 1, limit lower=0 upper=0 effort=0 velocity=0
- added joint joint57: type revolute, parent link56, child link57, origin xyz=56 0 0 rpy=0 0 0, axis 0 0 1, limit lower=0 upper=0 effort=0 velocity=0
- added joint joint58: type revolute, parent link57, child link58, origin xyz=57 0 0 rpy=0 0 0, axis 0 0 1, limit lower=0 upper=0 effort=0 velocity=0
- added joint joint59: type revolute, parent link58, child link59, origin xyz=58 0 0 rpy=0 0 0, axis 0 0 1, limit lower=0 upper=0 effort=0 velocity=0
- added joint joint60: type revolute, parent link59, child link60, origin xyz=59 0 0 rpy=0 0 0, axis 0 0 1, limit lower=0 upper=0 effort=0 velocity=0
- added joint joint61: type revolute, parent link60, child link61, origin xyz=60 0 0 rpy=0 0 0, axis 0 0 1, limit lower=0 upper=0 effort=0 velocity=0
- added joint joint62: type revolute, parent link61, child link62, origin xyz=61 0 0 rpy=0 0 0, axis 0 0 1, limit lower=0 upper=0 effort=0 velocity=0
- added joint joint63: type revolute, parent link62, child link63, origin xyz=62 0 0 rpy=0 0 0, axis 0 0 1, limit lower=0 upper=0 effort=0 velocity=0
- added joint joint64: type revolute, parent link63, child link64, origin xyz=63 0 0 rpy=0 0 0, axis 0 0 1, limit lower=0 upper=0 effort=0 velocity=0
- added joint joint65: type revolute, parent link64, child link65, origin xyz=64 0 0 rpy=0 0 0, axis 0 0 1, limit lower=0 upper=0 effort=0 velocity=0
- added joint joint66: type revolute, parent link65, child link66, origin xyz=65 0 0 rpy=0 0 0, axis 0 0 1, limit lower=0 upper=0 effort=0 velocity=0
- added joint joint67: type revolute, parent link66, child link67, origin xyz=66 0 0 rpy=0 0 0, axis 0 0 1, limit lower=0 upper=0 effort=0 velocity=0
- added joint joint68: type revolute, parent link67, child link68, origin xyz=67 0 0 rpy=0 0 0, axis 0 0 1, limit lower=0 upper=0 effort=0 velocity=0
- added joint joint69: type revolute, parent link68, child link69, origin xyz=68 0 0 rpy=0 0 0, axis 0 0 1, limit lower=0 upper=0 effort=0 velocity=0
- added joint joint70: type revolute, parent link69, child link70, origin xyz=69 0 0 rpy=0 0 0, axis 0 0 1, limit lower=0 upper=0 effort=0 velocity=0
- added joint joint71: type revolute, parent link70, child link71, origin xyz=70 0 0 rpy=0 0 0, axis 0 0 1, limit lower=0 upper=0 effort=0 velocity=0
- added joint joint72: type revolute, parent link71, child link72, origin xyz=71 0 0 rpy=0 0 0, axis 0 0 1, limit lower=0 upper=0 effort=0 velocity=0
- added joint joint73: type revolute, parent link72, child link73, origin xyz=72 0 0 rpy=0 0 0, axis 0 0 1, limit lower=0 upper=0 effort=0 velocity=0
- added joint joint74: type revolute, parent link73, child link74, origin xyz=73 0 0 rpy=0 0 0, axis 0 0 1, limit lower=0 upper=0 effort=0 velocity=0
- added joint joint75: type revolute, parent link74, child link75, origin xyz=74 0 0 rpy=0 0 0, axis 0 0 1, limit lower=0 upper=0 effort=0 velocity=0
- added joint joint76: type revolute, parent link75, child link76, origin xyz=75 0 0 rpy=0 0 0, axis 0 0 1, limit lower=0 upper=0 effort=0 velocity=0
- added joint joint77: type revolute, parent link76, child link77, origin xyz=76 0 0 rpy=0 0 0, axis 0 0 1, limit lower=0 upper=0 effort=0 velocity=0
- added joint joint78: type revolute, parent link77, child link78, origin xyz=77 0 0 rpy=0 0 0, axis 0 0 1, limit lower=0 upper=0 effort=0 velocity=0
- added joint joint79: type revolute, parent link78, child link79, origin xyz=78 0 0 rpy=0 0 0, axis 0 0 1, limit lower=0 upper=0 effort=0 velocity=0
- added joint joint80: type revolute, parent link79, child link80, origin xyz=79 0 0 rpy=0 0 0, axis 0 0 1, limit lower=0 upper=0 effort=0 velocity=0
