Commit message: generating more URDFS

File: 95link_bf_2.urdf (robot description, URDF)
Before this commit: robot 65link_bf_5, 66 links, 65 joints
Links:
- added link link66, mass 1.5
- added link link67, mass 1.5
- added link link68, mass 1.5
- added link link69, mass 1.5
- added link link70, mass 1.5
- added link link71, mass 1.5
- added link link72, mass 1.5
- added link link73, mass 1.5
- added link link74, mass 1.5
- added link link75, mass 1.5
- added link link76, mass 1.5
- added link link77, mass 1.5
- added link link78, mass 1.5
- added link link79, mass 1.5
- added link link80, mass 1.5
- added link link81, mass 1.5
- added link link82, mass 1.5
- added link link83, mass 1.5
- added link link84, mass 1.5
- added link link85, mass 1.5
- added link link86, mass 1.5
- added link link87, mass 1.5
- added link link88, mass 1.5
- added link link89, mass 1.5
- added link link90, mass 1.5
- added link link91, mass 1.5
- added link link92, mass 1.5
- added link link93, mass 1.5
- added link link94, mass 1.5
- added link link95, mass 1.5
Joints:
- added joint joint66: type revolute, parent link33, child link66, origin xyz=33 0 0 rpy=0 0 0, axis 0 0 1, limit lower=0 upper=0 effort=0 velocity=0
- added joint joint67: type revolute, parent link33, child link67, origin xyz=33 0 0 rpy=0 0 0, axis 0 0 1, limit lower=0 upper=0 effort=0 velocity=0
- added joint joint68: type revolute, parent link34, child link68, origin xyz=34 0 0 rpy=0 0 0, axis 0 0 1, limit lower=0 upper=0 effort=0 velocity=0
- added joint joint69: type revolute, parent link34, child link69, origin xyz=34 0 0 rpy=0 0 0, axis 0 0 1, limit lower=0 upper=0 effort=0 velocity=0
- added joint joint70: type revolute, parent link35, child link70, origin xyz=35 0 0 rpy=0 0 0, axis 0 0 1, limit lower=0 upper=0 effort=0 velocity=0
- added joint joint71: type revolute, parent link35, child link71, origin xyz=35 0 0 rpy=0 0 0, axis 0 0 1, limit lower=0 upper=0 effort=0 velocity=0
- added joint joint72: type revolute, parent link36, child link72, origin xyz=36 0 0 rpy=0 0 0, axis 0 0 1, limit lower=0 upper=0 effort=0 velocity=0
- added joint joint73: type revolute, parent link36, child link73, origin xyz=36 0 0 rpy=0 0 0, axis 0 0 1, limit lower=0 upper=0 effort=0 velocity=0
- added joint joint74: type revolute, parent link37, child link74, origin xyz=37 0 0 rpy=0 0 0, axis 0 0 1, limit lower=0 upper=0 effort=0 velocity=0
- added joint joint75: type revolute, parent link37, child link75, origin xyz=37 0 0 rpy=0 0 0, axis 0 0 1, limit lower=0 upper=0 effort=0 velocity=0
- added joint joint76: type revolute, parent link38, child link76, origin xyz=38 0 0 rpy=0 0 0, axis 0 0 1, limit lower=0 upper=0 effort=0 velocity=0
- added joint joint77: type revolute, parent link38, child link77, origin xyz=38 0 0 rpy=0 0 0, axis 0 0 1, limit lower=0 upper=0 effort=0 velocity=0
- added joint joint78: type revolute, parent link39, child link78, origin xyz=39 0 0 rpy=0 0 0, axis 0 0 1, limit lower=0 upper=0 effort=0 velocity=0
- added joint joint79: type revolute, parent link39, child link79, origin xyz=39 0 0 rpy=0 0 0, axis 0 0 1, limit lower=0 upper=0 effort=0 velocity=0
- added joint joint80: type revolute, parent link40, child link80, origin xyz=40 0 0 rpy=0 0 0, axis 0 0 1, limit lower=0 upper=0 effort=0 velocity=0
- added joint joint81: type revolute, parent link40, child link81, origin xyz=40 0 0 rpy=0 0 0, axis 0 0 1, limit lower=0 upper=0 effort=0 velocity=0
- added joint joint82: type revolute, parent link41, child link82, origin xyz=41 0 0 rpy=0 0 0, axis 0 0 1, limit lower=0 upper=0 effort=0 velocity=0
- added joint joint83: type revolute, parent link41, child link83, origin xyz=41 0 0 rpy=0 0 0, axis 0 0 1, limit lower=0 upper=0 effort=0 velocity=0
- added joint joint84: type revolute, parent link42, child link84, origin xyz=42 0 0 rpy=0 0 0, axis 0 0 1, limit lower=0 upper=0 effort=0 velocity=0
- added joint joint85: type revolute, parent link42, child link85, origin xyz=42 0 0 rpy=0 0 0, axis 0 0 1, limit lower=0 upper=0 effort=0 velocity=0
- added joint joint86: type revolute, parent link43, child link86, origin xyz=43 0 0 rpy=0 0 0, axis 0 0 1, limit lower=0 upper=0 effort=0 velocity=0
- added joint joint87: type revolute, parent link43, child link87, origin xyz=43 0 0 rpy=0 0 0, axis 0 0 1, limit lower=0 upper=0 effort=0 velocity=0
- added joint joint88: type revolute, parent link44, child link88, origin xyz=44 0 0 rpy=0 0 0, axis 0 0 1, limit lower=0 upper=0 effort=0 velocity=0
- added joint joint89: type revolute, parent link44, child link89, origin xyz=44 0 0 rpy=0 0 0, axis 0 0 1, limit lower=0 upper=0 effort=0 velocity=0
- added joint joint90: type revolute, parent link45, child link90, origin xyz=45 0 0 rpy=0 0 0, axis 0 0 1, limit lower=0 upper=0 effort=0 velocity=0
- added joint joint91: type revolute, parent link45, child link91, origin xyz=45 0 0 rpy=0 0 0, axis 0 0 1, limit lower=0 upper=0 effort=0 velocity=0
- added joint joint92: type revolute, parent link46, child link92, origin xyz=46 0 0 rpy=0 0 0, axis 0 0 1, limit lower=0 upper=0 effort=0 velocity=0
- added joint joint93: type revolute, parent link46, child link93, origin xyz=46 0 0 rpy=0 0 0, axis 0 0 1, limit lower=0 upper=0 effort=0 velocity=0
- added joint joint94: type revolute, parent link47, child link94, origin xyz=47 0 0 rpy=0 0 0, axis 0 0 1, limit lower=0 upper=0 effort=0 velocity=0
- added joint joint95: type revolute, parent link47, child link95, origin xyz=47 0 0 rpy=0 0 0, axis 0 0 1, limit lower=0 upper=0 effort=0 velocity=0
- joint joint10: origin xyz=2 0 0 rpy=0 0 0 -> xyz=5 0 0 rpy=0 0 0; parent link2 -> link5
- joint joint11: origin xyz=2 0 0 rpy=0 0 0 -> xyz=5 0 0 rpy=0 0 0; parent link2 -> link5
- joint joint12: origin xyz=3 0 0 rpy=0 0 0 -> xyz=6 0 0 rpy=0 0 0; parent link3 -> link6
- joint joint13: origin xyz=3 0 0 rpy=0 0 0 -> xyz=6 0 0 rpy=0 0 0; parent link3 -> link6
- joint joint14: origin xyz=3 0 0 rpy=0 0 0 -> xyz=7 0 0 rpy=0 0 0; parent link3 -> link7
- joint joint15: origin xyz=3 0 0 rpy=0 0 0 -> xyz=7 0 0 rpy=0 0 0; parent link3 -> link7
- joint joint16: origin xyz=3 0 0 rpy=0 0 0 -> xyz=8 0 0 rpy=0 0 0; parent link3 -> link8
- joint joint17: origin xyz=4 0 0 rpy=0 0 0 -> xyz=8 0 0 rpy=0 0 0; parent link4 -> link8
- joint joint18: origin xyz=4 0 0 rpy=0 0 0 -> xyz=9 0 0 rpy=0 0 0; parent link4 -> link9
- joint joint19: origin xyz=4 0 0 rpy=0 0 0 -> xyz=9 0 0 rpy=0 0 0; parent link4 -> link9
- joint joint20: origin xyz=4 0 0 rpy=0 0 0 -> xyz=10 0 0 rpy=0 0 0; parent link4 -> link10
- joint joint21: origin xyz=4 0 0 rpy=0 0 0 -> xyz=10 0 0 rpy=0 0 0; parent link4 -> link10
- joint joint22: origin xyz=5 0 0 rpy=0 0 0 -> xyz=11 0 0 rpy=0 0 0; parent link5 -> link11
- joint joint23: origin xyz=5 0 0 rpy=0 0 0 -> xyz=11 0 0 rpy=0 0 0; parent link5 -> link11
- joint joint24: origin xyz=5 0 0 rpy=0 0 0 -> xyz=12 0 0 rpy=0 0 0; parent link5 -> link12
- joint joint25: origin xyz=5 0 0 rpy=0 0 0 -> xyz=12 0 0 rpy=0 0 0; parent link5 -> link12
- joint joint26: origin xyz=5 0 0 rpy=0 0 0 -> xyz=13 0 0 rpy=0 0 0; parent link5 -> link13
- joint joint27: origin xyz=6 0 0 rpy=0 0 0 -> xyz=13 0 0 rpy=0 0 0; parent link6 -> link13
- joint joint28: origin xyz=6 0 0 rpy=0 0 0 -> xyz=14 0 0 rpy=0 0 0; parent link6 -> link14
- joint joint29: origin xyz=6 0 0 rpy=0 0 0 -> xyz=14 0 0 rpy=0 0 0; parent link6 -> link14
- joint joint30: origin xyz=6 0 0 rpy=0 0 0 -> xyz=15 0 0 rpy=0 0 0; parent link6 -> link15
- joint joint31: origin xyz=6 0 0 rpy=0 0 0 -> xyz=15 0 0 rpy=0 0 0; parent link6 -> link15
- joint joint32: origin xyz=7 0 0 rpy=0 0 0 -> xyz=16 0 0 rpy=0 0 0; parent link7 -> link16
- joint joint33: origin xyz=7 0 0 rpy=0 0 0 -> xyz=16 0 0 rpy=0 0 0; parent link7 -> link16
- joint joint34: origin xyz=7 0 0 rpy=0 0 0 -> xyz=17 0 0 rpy=0 0 0; parent link7 -> link17
- joint joint35: origin xyz=7 0 0 rpy=0 0 0 -> xyz=17 0 0 rpy=0 0 0; parent link7 -> link17
- joint joint36: origin xyz=7 0 0 rpy=0 0 0 -> xyz=18 0 0 rpy=0 0 0; parent link7 -> link18
- joint joint37: origin xyz=8 0 0 rpy=0 0 0 -> xyz=18 0 0 rpy=0 0 0; parent link8 -> link18
- joint joint38: origin xyz=8 0 0 rpy=0 0 0 -> xyz=19 0 0 rpy=0 0 0; parent link8 -> link19
- joint joint39: origin xyz=8 0 0 rpy=0 0 0 -> xyz=19 0 0 rpy=0 0 0; parent link8 -> link19
- joint joint4: origin xyz=1 0 0 rpy=0 0 0 -> xyz=2 0 0 rpy=0 0 0; parent link1 -> link2
- joint joint40: origin xyz=8 0 0 rpy=0 0 0 -> xyz=20 0 0 rpy=0 0 0; parent link8 -> link20
- joint joint41: origin xyz=8 0 0 rpy=0 0 0 -> xyz=20 0 0 rpy=0 0 0; parent link8 -> link20
- joint joint42: origin xyz=9 0 0 rpy=0 0 0 -> xyz=21 0 0 rpy=0 0 0; parent link9 -> link21
- joint joint43: origin xyz=9 0 0 rpy=0 0 0 -> xyz=21 0 0 rpy=0 0 0; parent link9 -> link21
- joint joint44: origin xyz=9 0 0 rpy=0 0 0 -> xyz=22 0 0 rpy=0 0 0; parent link9 -> link22
- joint joint45: origin xyz=9 0 0 rpy=0 0 0 -> xyz=22 0 0 rpy=0 0 0; parent link9 -> link22
- joint joint46: origin xyz=9 0 0 rpy=0 0 0 -> xyz=23 0 0 rpy=0 0 0; parent link9 -> link23
- joint joint47: origin xyz=10 0 0 rpy=0 0 0 -> xyz=23 0 0 rpy=0 0 0; parent link10 -> link23
- joint joint48: origin xyz=10 0 0 rpy=0 0 0 -> xyz=24 0 0 rpy=0 0 0; parent link10 -> link24
- joint joint49: origin xyz=10 0 0 rpy=0 0 0 -> xyz=24 0 0 rpy=0 0 0; parent link10 -> link24
- joint joint5: origin xyz=1 0 0 rpy=0 0 0 -> xyz=2 0 0 rpy=0 0 0; parent link1 -> link2
- joint joint50: origin xyz=10 0 0 rpy=0 0 0 -> xyz=25 0 0 rpy=0 0 0; parent link10 -> link25
- joint joint51: origin xyz=10 0 0 rpy=0 0 0 -> xyz=25 0 0 rpy=0 0 0; parent link10 -> link25
- joint joint52: origin xyz=11 0 0 rpy=0 0 0 -> xyz=26 0 0 rpy=0 0 0; parent link11 -> link26
- joint joint53: origin xyz=11 0 0 rpy=0 0 0 -> xyz=26 0 0 rpy=0 0 0; parent link11 -> link26
- joint joint54: origin xyz=11 0 0 rpy=0 0 0 -> xyz=27 0 0 rpy=0 0 0; parent link11 -> link27
- joint joint55: origin xyz=11 0 0 rpy=0 0 0 -> xyz=27 0 0 rpy=0 0 0; parent link11 -> link27
- joint joint56: origin xyz=11 0 0 rpy=0 0 0 -> xyz=28 0 0 rpy=0 0 0; parent link11 -> link28
- joint joint57: origin xyz=12 0 0 rpy=0 0 0 -> xyz=28 0 0 rpy=0 0 0; parent link12 -> link28
- joint joint58: origin xyz=12 0 0 rpy=0 0 0 -> xyz=29 0 0 rpy=0 0 0; parent link12 -> link29
- joint joint59: origin xyz=12 0 0 rpy=0 0 0 -> xyz=29 0 0 rpy=0 0 0; parent link12 -> link29
- joint joint6: origin xyz=1 0 0 rpy=0 0 0 -> xyz=3 0 0 rpy=0 0 0; parent link1 -> link3
- joint joint60: origin xyz=12 0 0 rpy=0 0 0 -> xyz=30 0 0 rpy=0 0 0; parent link12 -> link30
- joint joint61: origin xyz=12 0 0 rpy=0 0 0 -> xyz=30 0 0 rpy=0 0 0; parent link12 -> link30
- joint joint62: origin xyz=13 0 0 rpy=0 0 0 -> xyz=31 0 0 rpy=0 0 0; parent link13 -> link31
- joint joint63: origin xyz=13 0 0 rpy=0 0 0 -> xyz=31 0 0 rpy=0 0 0; parent link13 -> link31
- joint joint64: origin xyz=13 0 0 rpy=0 0 0 -> xyz=32 0 0 rpy=0 0 0; parent link13 -> link32
- joint joint65: origin xyz=13 0 0 rpy=0 0 0 -> xyz=32 0 0 rpy=0 0 0; parent link13 -> link32
- joint joint7: origin xyz=2 0 0 rpy=0 0 0 -> xyz=3 0 0 rpy=0 0 0; parent link2 -> link3
- joint joint8: origin xyz=2 0 0 rpy=0 0 0 -> xyz=4 0 0 rpy=0 0 0; parent link2 -> link4
- joint joint9: origin xyz=2 0 0 rpy=0 0 0 -> xyz=4 0 0 rpy=0 0 0; parent link2 -> link4
